File: XShiftGenerator.sch (KiCad schematic (older format))
At the start: 6 parts, among them U10 LM358

Commit message: Fixed some bugs, finished block symbols
Parts:
- RV4: footprint Potentiometer_THT:Potentiometer_Bourns_3299W_Vertical -> Potentiometer_THT:Potentiometer_Bourns_3296W_Vertical
Changed lines of the file:
@@
 encoding utf-8
 Sheet 12 13
-Title ""
-Date ""
-Rev ""
-Comp ""
+Title "Horiznontal Shift Generator"
+Date "2021-04-20"
+Rev "2.0"
+Comp "Filip Piórski"
 Comment1 ""
 Comment2 ""
@@
 F 0 "RV4" V 5100 3400 50  0000 R CNN
 F 1 "1k" V 5100 3600 50  0000 R CNN
-F 2 "Potentiometer_THT:Potentiometer_Bourns_3299W_Vertical" H 5200 3450 50  0001 C CNN
+F 2 "Potentiometer_THT:Potentiometer_Bourns_3296W_Vertical" H 5200 3450 50  0001 C CNN
 F 3 "~" H 5200 3450 50  0001 C CNN
 	1    5200 3450
